File: PCB_Project.kicad_sch (KiCad schematic)
At the start: 0 parts

Commit message: Add files via upload
Parts:
- added D1, D2, D3: L08R5000Q1, L08R5000Q1:LEDRD254W57D500H1070, symbol L08R5000Q1:L08R5000Q1
- added R1, R2, R3: R, symbol Device:R
- added SW1, SW2, SW3: SW_Push, symbol Switch:SW_Push
- added U1: XIAO-RP2040-DIP, Module:MOUDLE14P-XIAO-DIP-SMD, symbol Seeed_Studio_XIAO_Series:XIAO-RP2040-DIP
Connections:
- new net: D3.A, R3.1
- new net: D1.A, R1.1
- new net: D2.A, R2.1
- new net Button1: SW1.1, U1.1 (GPIO26/ADC0/A0)
- new net Button2: SW2.1, U1.2 (GPIO27/ADC1/A1)
- new net Button3: SW3.1, U1.3 (GPIO28/ADC2/A2)
- new net GND: U1.13 (GND)
- new net LED1: R1.2, U1.4 (GPIO29/ADC3/A3)
- new net LED2: R2.2, U1.5 (GPIO6/SDA)
- new net LED3: R3.2, U1.6 (GPIO7/SCL)

Commit message: Add files via upload
Parts:
- D1, D2, D3: footprint L08R5000Q1:LEDRD254W57D500H1070 -> footprints:LEDRD254W57D500H1070
- R1, R2, R3: footprint (none) -> Resistor_THT:R_Axial_DIN0204_L3.6mm_D1.6mm_P5.08mm_Horizontal
- SW1, SW2, SW3: footprint (none) -> Button_Switch_Keyboard:SW_Cherry_MX_1.00u_PCB
- U1: footprint Module:MOUDLE14P-XIAO-DIP-SMD -> footprints:XIAO-RP2040-DIP
Connections:
- net GND: now also D1.C, D2.C, D3.C, SW1.2, SW2.2, SW3.2
